Commit message: replaced launcher files with correct ones

File: launch/simple_world.urdf (robot description, URDF)
Before this commit: robot test, 8 links, 7 joints
Links:
- added link obs_7, mass 1000.0; collision box size=0.4 0.4 0.2; visual box size=0.4 0.4 0.2
- added link obs_8, mass 1000.0; collision box size=0.05 0.05 0.15; visual box size=0.05 0.05 0.15
- added link obs_9, mass 1000.0; collision box size=0.05 0.05 0.15; visual box size=0.05 0.05 0.15
- added link obs_top, mass 1000.0; collision box size=0.05 0.25 0.05; visual box size=0.05 0.25 0.05
Joints:
- added joint join10: type fixed, parent wall_1, child obs_7, origin xyz=0.6 0 0.1 rpy=0 0 0
- added joint join11: type fixed, parent wall_1, child obs_8, origin xyz=0.5 0.1 0.275 rpy=0 0 0
- added joint join12: type fixed, parent wall_1, child obs_9, origin xyz=0.5 -0.1 0.275 rpy=0 0 0
- added joint join13: type fixed, parent wall_1, child obs_top, origin xyz=0.5 0 0.375 rpy=0 0 0
